File: Sensor_hw/Sensor.kicad_pcb (KiCad board)
At the start: 2 copper layers, 29 x 32.5 mm, 18 parts, among them Q1 TSOP48xx, Q2 TSOP48xx, Q3 TSOP48xx, Q4 WS2812B

Commit message: + Head started
Parts:
- moved XL1 2.85 mm to (138.2, 108.8)
- moved XL2 0.10 mm to (161.5, 108.8)
Other:
- outline, holes or cut-outs redrawn
Changed lines of the file:
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@@
     (links 34)
     (no_connects 0)
-    (area 133.949999 88.699999 163.050001 121.300001)
+    (area 132.66635 88.25 163.500001 121.750001)
     (thickness 1.6)
-    (drawings 27)
+    (drawings 31)
     (tracks 271)
     (zones 0)
@@
   (page A4)
   (layers
-    (0 F.Cu signal)
-    (31 B.Cu signal)
+    (0 F.Cu signal hide)
+    (31 B.Cu signal hide)
     (36 B.SilkS user)
     (37 F.SilkS user)
     (38 B.Mask user)
     (39 F.Mask user)
-    (40 Dwgs.User user hide)
+    (40 Dwgs.User user)
     (44 Edge.Cuts user)
   )
@@
     (pad_to_mask_clearance 0.2)
     (aux_axis_origin 0 0)
-    (visible_elements 7FFFF77F)
+    (visible_elements 7FFFF75F)
     (pcbplotparams
       (layerselection 0x00030_80000001)
@@
   )
   (module Connectors:PLS-4 (layer F.Cu)
-    (at 135.4 108.8 90)
+    (at 138.25 108.83 90)
     (descr "Single-line connector 4-pin")
     (fp_text reference XL1 (at -0.7 1.85 90) (layer F.SilkS)
@@
   )
   (module Connectors:PLS-4 (layer F.Cu)
-    (at 161.6 108.8 90)
+    (at 161.5 108.8 90)
     (descr "Single-line connector 4-pin")
     (fp_text reference XL2 (at -0.8 -1.8 90) (layer F.SilkS)
@@
     )
   )
+  (gr_circle (center 136 100.5) (end 137 100.5) (layer Edge.Cuts) (width 0.1))
+  (gr_circle (center 136 109.5) (end 137 109.5) (layer Edge.Cuts) (width 0.1))
+  (gr_circle (center 136 106.5) (end 137 106.5) (layer Edge.Cuts) (width 0.1))
+  (gr_circle (center 136 103.5) (end 137 103.5) (layer Edge.Cuts) (width 0.1))
   (gr_line (start 137 116.75) (end 134 113) (angle 90) (layer Edge.Cuts) (width 0.1))
   (gr_line (start 140.75 119.5) (end 137 116.75) (angle 90) (layer Edge.Cuts) (width 0.1))

Commit message: + Sensor sent to manufacture * Head: barrel socket is here + armlet case
Parts:
- removed HOLE2: HOLE_METALLED, PCB:Hole3d3_out5d5mm
- added XL3: CONN_1, PCB:Oval6x3, B.Cu at (144.0, 100.0)
- added XL4: CONN_1, PCB:Oval6x3, B.Cu at (142.0, 94.5)
- added XL5: CONN_1, PCB:Oval6x3, B.Cu at (156.0, 116.2)
- added XL6: CONN_1, PCB:Oval6x3, B.Cu at (154.5, 112.0)
- added XL7: CONN_1, PCB:Oval6x3, B.Cu at (153.0, 100.0)
- added XL8: CONN_1, PCB:Oval6x3, B.Cu at (155.0, 94.5)
- Q4: value WS2812B -> LED_RGB_WS2812B
- XL1, XL2: value CONN_4 -> CONN_1; footprint Connectors:PLS-4 -> PCB:Oval6x3; moved to B.Cu
- moved XL2 19.3 mm to (142.5, 112.0), turned to 330 degrees
- moved C4 15.2 mm to (153.8, 96.0)
- moved HOLE1 8.75 mm to (148.5, 105.0)
- moved XL1 7.91 mm to (141.0, 116.2), turned to 150 degrees
- moved Q4 6.13 mm to (148.5, 96.0), turned to 180 degrees
- moved D1 5.97 mm to (148.5, 115.5), turned to 90 degrees
- moved R4 4.90 mm to (143.5, 115.5)
- moved C5 0.80 mm to (141.0, 111.4)
- moved C2 0.05 mm to (153.8, 103.5)
- moved R2 0.05 mm to (153.8, 99.8)
Connections:
- XL2 pad 1: GND -> VCC
Routing:
- net /LED_DOUT: track 18.4 -> 5.24 mm, vias 0 -> 1
- net VCC: track 61.8 -> 48.8 mm, vias 2 -> 3
- net GND: track 159.4 -> 149.1 mm
- net /LED_DIN: track 8.78 -> 5.50 mm, vias 0 -> 1
- net Net-(D1-PadA): track 2.73 -> 5.13 mm
- net /SNS: track 39.6 -> 37.7 mm
Other:
- board size 29 x 32.5 mm -> 27 x 31 mm
- rule pad_to_mask_clearance: 0.2 -> 0.1
- board text added: "GND"
- board text added: "LED DIN"
- board text added: "LED DOUT"
- board text added: "SNS"
- board text added: "VCC"
