File: GunRadio_hw/GunRadio.kicad_pcb (KiCad board)
At the start: 2 copper layers, 24.4 x 61.7 mm, 41 parts

Commit message: + GunRadio nears completion
Parts:
- ANT1: footprint Radio:ANT_868_MEANDER_4HOR_35mm -> Radio:ANT_868_GunRADIO
- moved XL3 83.1 mm to (135.4, 155.8)
- moved D1 80.9 mm to (140.0, 143.4), turned to 270 degrees
- moved ANT1 79.5 mm to (139.7, 96.1)
- moved C10 77.2 mm to (130.4, 128.8), turned to 90 degrees
- moved DA1 73.6 mm to (145.8, 153.8), turned to 270 degrees
- moved C12 66.2 mm to (139.2, 132.8), turned to 180 degrees
- moved C8 65.2 mm to (134.4, 119.7)
- moved C2 64.2 mm to (143.2, 153.8), turned to 90 degrees
- moved R1 63.2 mm to (140.0, 140.2), turned to 270 degrees
- moved R4 63.1 mm to (134.4, 103.3), turned to 180 degrees
- moved C5 61.6 mm to (134.4, 101.7), turned to 180 degrees
- moved XL1 61.4 mm to (129.0, 107.4), turned to 270 degrees
- moved C9 59.2 mm to (143.1, 99.3)
- moved R3 57.4 mm to (145.1, 107.8), turned to 90 degrees
- moved C6 57.1 mm to (139.2, 134.6), turned to 180 degrees
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Connections:
- DD1 pad 14: Net-(DD1-Pad14) -> (no net)
- DD1 pad 19: Net-(DD1-Pad19) -> (no net)
- DD1 pad 2: Net-(DD1-Pad2) -> (no net)
- DD1 pad 20: Net-(DD1-Pad20) -> (no net)
- DD1 pad 3: Net-(DD1-Pad3) -> (no net)
- DD1 pad 32: Net-(DD1-Pad32) -> (no net)
- DD1 pad 33: Net-(DD1-Pad33) -> (no net)
- DD1 pad 38: Net-(DD1-Pad38) -> (no net)
- DD1 pad 39: Net-(DD1-Pad39) -> (no net)
- DD1 pad 4: Net-(DD1-Pad4) -> (no net)
- DD1 pad 40: Net-(DD1-Pad40) -> (no net)
- DD1 pad 41: Net-(DD1-Pad41) -> (no net)
- DD1 pad 42: Net-(DD1-Pad42) -> (no net)
- DD1 pad 43: Net-(DD1-Pad43) -> (no net)
- DD1 pad 45: Net-(DD1-Pad45) -> (no net)
- DD1 pad 46: Net-(DD1-Pad46) -> (no net)
- XL1 pad 8: Net-(XL1-Pad8) -> GND
- XL4 pad 1: PwrMCU -> +3.3V
Routing:
- net GND: track 0.00 -> 115.4 mm, vias 0 -> 6
- net +3.3V: track 0.00 -> 106.6 mm, vias 0 -> 7
- net /UART_TX: track 0.00 -> 21.7 mm
- net /UART_RX: track 0.00 -> 21.7 mm
- net /CC_MOSI: track 0.00 -> 18.0 mm
- net Net-(DD1-Pad21): track 0.00 -> 16.7 mm
- net Net-(DD1-Pad22): track 0.00 -> 16.0 mm
- net Net-(C4-Pad1): track 0.00 -> 12.0 mm
- net Net-(DD1-Pad25): track 0.00 -> 11.9 mm
- net /CC_GDO2: track 0.00 -> 10.6 mm
- net Net-(DD1-Pad26): track 0.00 -> 10.2 mm
- net /CC_GDO0: track 0.00 -> 10.00 mm
- net Net-(C17-Pad1): track 0.00 -> 9.55 mm
- net Net-(DD1-Pad27): track 0.00 -> 8.41 mm
- net Net-(C18-Pad1): track 0.00 -> 7.79 mm
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Other:
- board size 24.4 x 61.7 mm -> 24.4 x 77.7 mm
- net class Default: trace_width 0.25 -> 0.2; via_dia 0.6 -> 0.9
- net class Wide added: clearance 0.2, trace_width 0.5, via_dia 0.9, via_drill 0.4

Commit message: GunRadio finished
Parts:
- moved R2 0.20 mm to (145.4, 125.5)
Routing:
- net GND: track 115.4 -> 427.8 mm, vias 6 -> 106
- net +3.3V: track 106.6 -> 167.1 mm, vias 7 -> 12
- net /Trigger: track 0.00 -> 34.1 mm, vias 0 -> 3
- net Net-(DD1-Pad10): track 0.00 -> 33.3 mm, vias 0 -> 2
- net /UART_TX: track 21.7 -> 46.9 mm, vias 0 -> 2
- net /UART_RX: track 21.7 -> 44.1 mm, vias 0 -> 1
- net /SWDIO: track 0.00 -> 20.0 mm, vias 0 -> 1
- net /CC_SCK: track 0.00 -> 18.2 mm
- net Net-(DD1-Pad18): track 0.00 -> 17.9 mm, vias 0 -> 2
- net /CC_MISO: track 0.00 -> 17.9 mm, vias 0 -> 2
- net /CC_CS: track 6.26 -> 23.4 mm
- net /SWCLK: track 0.00 -> 11.8 mm
- net /CC_GDO0: track 10.00 -> 20.0 mm, vias 0 -> 2
- net /CC_GDO2: track 10.6 -> 20.1 mm
- net Net-(D1-PadA): track 0.00 -> 1.69 mm
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- added copper zone on B.Cu, net GND
- added copper zone on F.Cu, net GND
